Commit message: Fixed name of link to make it consistent with the model used by Drake.

File: drake_cars_examples/models/drake_prius/xacro/drake_prius_base.xacro (robot description, xacro)
@@ -311,5 +311,5 @@
     </visual>
   </link>
-  <link name="chassis">
+  <link name="body">
     <inertial>
       <mass value="5.42794"/>
@@ -403,5 +403,5 @@
   <joint name="chassis" type="fixed">
     <parent link="chassis_floor"/>
-    <child link="chassis"/>
+    <child link="body"/>
     <origin rpy="0  0  0" xyz="0 0 0.006857999999999975226927518"/>
     <axis xyz="0  0  0"/>
